File: BSidesCBR2019.kicad_pcb (KiCad board)
At the start: 2 copper layers, 44.9 x 114.1 mm, 26 parts, among them J1 SAO, J2 LSAO, J3 CONN_01X08, SW1 RESET, SW3 <<, SW4 O, SW5 >>, U1 ATMEGA328P-AU, U2 Nokia_5110_LCD, Y1 16Mhz

Commit message: Added footprints and models, v8 gerbs
Parts:
- renumbered POWER to SW2
Connections:
- SW3 pad 1: +3.3v -> GND
- SW4 pad 1: +3.3v -> GND
- SW5 pad 1: +3.3v -> GND
Routing:
- net GND: track 20.8 -> 38.0 mm, vias 6 -> 9
Changed lines of the file:
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@@
     (thickness 1.6)
     (drawings 103)
-    (tracks 360)
+    (tracks 368)
     (zones 0)
     (modules 26)
@@
     (visible_elements FFFFFF7F)
     (pcbplotparams
-      (layerselection 0x010f0_80000001)
+      (layerselection 0x010f0_ffffffff)
       (usegerberextensions false)
       (usegerberattributes false)
@@
     (descr "Ultraminiature Surface Mount Slide Switch")
     (attr smd)
-    (fp_text reference POWER (at 0 3.2) (layer B.SilkS)
+    (fp_text reference SW2 (at 0 3.2) (layer B.Fab)
       (effects (font (size 1 1) (thickness 0.15)) (justify mirror))
     )
@@
       (effects (font (size 1 1) (thickness 0.15)) (justify mirror))
     )
-    (fp_text user POWAH (at 0 3.2) (layer B.Fab)
+    (fp_text user POWER (at 0.127 3.5306) (layer B.SilkS)
       (effects (font (size 1 1) (thickness 0.15)) (justify mirror))
     )
@@
     (pad "" smd rect (at 3.65 0.78) (size 1 0.8) (layers B.Cu B.Paste B.Mask))
     (pad "" smd rect (at -3.65 0.78) (size 1 0.8) (layers B.Cu B.Paste B.Mask))
-    (model /home/user/Boards/BSidesCBR2019/3d/switch_kps-1290-k.wrl
+    (model ./3d/switch_kps-1290-k.wrl
       (at (xyz 0 0 0))
       (scale (xyz 1 1 1))
@@
     (fp_line (start -3.1 3.25) (end -3.1 -3.25) (layer F.Fab) (width 0.1))
     (pad 1 smd rect (at -2.875 -2 90) (size 2.75 1) (layers F.Cu F.Paste F.Mask)
-      (net 4 +3.3v))
+      (net 1 GND))
     (pad 1 smd rect (at 2.875 -2 90) (size 2.75 1) (layers F.Cu F.Paste F.Mask)
-      (net 4 +3.3v))
+      (net 1 GND))
     (pad 2 smd rect (at 2.875 2 90) (size 2.75 1) (layers F.Cu F.Paste F.Mask)
       (net 32 BUTTONL))
@@
     (fp_line (start -3.1 3.25) (end -3.1 -3.25) (layer F.Fab) (width 0.1))
     (pad 1 smd rect (at -2.875 -2 90) (size 2.75 1) (layers F.Cu F.Paste F.Mask)
-      (net 4 +3.3v))
+      (net 1 GND))
     (pad 1 smd rect (at 2.875 -2 90) (size 2.75 1) (layers F.Cu F.Paste F.Mask)
-      (net 4 +3.3v))
+      (net 1 GND))
     (pad 2 smd rect (at 2.875 2 90) (size 2.75 1) (layers F.Cu F.Paste F.Mask)
       (net 33 BUTTONOK))
@@
     (fp_line (start -3.1 3.25) (end -3.1 -3.25) (layer F.Fab) (width 0.1))
     (pad 1 smd rect (at -2.875 -2 90) (size 2.75 1) (layers F.Cu F.Paste F.Mask)
-      (net 4 +3.3v))
+      (net 1 GND))
     (pad 1 smd rect (at 2.875 -2 90) (size 2.75 1) (layers F.Cu F.Paste F.Mask)
-      (net 4 +3.3v))
+      (net 1 GND))
     (pad 2 smd rect (at 2.875 2 90) (size 2.75 1) (layers F.Cu F.Paste F.Mask)
       (net 34 BUTTONR))
@@
   (segment (start 49.13 96.27) (end 48.98 96.27) (width 0.3) (layer B.Cu) (net 1) (status 30))
   (via (at 78.03 85.17) (size 0.6) (drill 0.4) (layers F.Cu B.Cu) (net 1))
+  (segment (start 48.0888 117.6844) (end 48.0888 113.6094) (width 0.3) (layer F.Cu) (net 1))
+  (segment (start 48.0888 119.3594) (end 48.0888 117.6844) (width 0.3) (layer F.Cu) (net 1))
+  (segment (start 56.9468 117.7558) (end 56.9468 113.6808) (width 0.3) (layer F.Cu) (net 1))
+  (segment (start 56.9468 119.4308) (end 56.9468 117.7558) (width 0.3) (layer F.Cu) (net 1))
+  (segment (start 65.9384 119.2276) (end 65.9384 113.4776) (width 0.3) (layer F.Cu) (net 1))
+  (via (at 65.9384 113.4776) (size 0.6) (drill 0.4) (layers F.Cu B.Cu) (net 1))
+  (via (at 56.9468 113.6808) (size 0.6) (drill 0.4) (layers F.Cu B.Cu) (net 1))
+  (via (at 48.0888 119.3594) (size 0.6) (drill 0.4) (layers F.Cu B.Cu) (net 1))
   (segment (start 40.54 83.5) (end 43.71 83.5) (width 0.3) (layer F.Cu) (net 2))
   (segment (start 43.71 83.5) (end 44.02 83.19) (width 0.3) (layer F.Cu) (net 2))
