File: BSidesCBR2019.sch (KiCad schematic (older format))
At the start: 35 parts, among them IC1 Si4455-B1A-FM, J1 SAO, J2 LSAO, SW1 RESET, U1 ATMEGA328P-AU, U2 Nokia_5110_LCD, Y1 16Mhz, Y2 30Mhz

Commit message: Added each gerber revision, updated with latest version of board designs.
Parts:
- removed AE1: Antenna_Dipole, dipole:ti-dn023-antenna, symbol Antenna_Dipole
- removed C0, C2, C3, C4, CM1, CM2, CM3, CR1, CR2: (no value), Capacitors_SMD:C_0805_HandSoldering, symbol C_Small
- removed D5: 1N4148, Diodes_SMD:D_SOD-323_HandSoldering, symbol D
- removed IC1: Si4455-B1A-FM, Si4455-B1A-FM:QFN50P300X300X80-21N-D, symbol Si4455-B1A-FM
- removed L0, LM1, LM2, LR1, LR2, Lchoke1: (no value), Inductors_SMD:L_0805_HandSoldering, symbol L_Small
- removed ROC1: (no value), Resistors_SMD:R_0805_HandSoldering, symbol R_Small
- removed Y2: 30Mhz, Crystals:Resonator_SMD-3pin_7.2x3.0mm_HandSoldering, symbol Crystal_GND2
- added D3, D4: BL, LEDs:LED_0603, symbol LED_Small
- added J3: CONN_01X08, Pin_Headers:Pin_Header_Straight_1x08_Pitch2.54mm, symbol CONN_01X08
- added R6: LR, Resistors_SMD:R_0805_HandSoldering, symbol R_Small
- added R7, R8: 1k, Resistors_SMD:R_0805_HandSoldering, symbol R_Small
- added R9: 1K, Resistors_SMD:R_0805_HandSoldering, symbol R_Small
- added SW2: SW_SPST, Buttons_Switches_SMD:SW_SPDT_PCM12, symbol SW_SPDT
- added SW3: <<, Buttons_Switches_SMD:SW_SPST_B3SL-1002P, symbol SW_Push
- added SW4: O, Buttons_Switches_SMD:SW_SPST_B3SL-1002P, symbol SW_Push
- added SW5: >>, Buttons_Switches_SMD:SW_SPST_B3SL-1002P, symbol SW_Push
- C1: value (none) -> 100n
- D1, D2: footprint LEDs:LED_0805_HandSoldering -> LEDs:LED_0603
- R3: value 1K -> LR
- R4: value 1M -> 10K
- Y1: footprint Crystals:Resonator_SMD-3pin_7.2x3.0mm_HandSoldering -> Crystals:Crystal_SMD_TXC_7M-4pin_3.2x2.5mm_HandSoldering; symbol Crystal_GND2 -> Crystal_GND24
Connections:
- net labels added: A6, A7, AD0, AD1, AD2, AD3, BAT+, BUTTONS, D10, D3, D4, D9, OSC, VOUT
- net labels removed: RFNIRQ, RFNSEL, RXN, RXP, TXA, XIN, XOUT
- wire segments 120 -> 115
Other:
- moved on the sheet: BT1, D1, R1, R5

Commit message: Fixes for buttons, added more silkscreen
Parts:
- removed R7, R8: 1k, Resistors_SMD:R_0805_HandSoldering, symbol R_Small
- removed R9: 1K, Resistors_SMD:R_0805_HandSoldering, symbol R_Small
- BT1: symbol Battery_Cell_PWR -> BSidesCBR2019-rescue:Battery_Cell_PWR
- C1: symbol C_Small -> BSidesCBR2019-rescue:C_Small
- D1, D2, D3, D4: symbol LED_Small -> BSidesCBR2019-rescue:LED_Small
- J1: symbol Conn_02x02_Odd_Even -> BSidesCBR2019-rescue:Conn_02x02_Odd_Even
- J2: symbol Conn_02x03_Odd_Even -> BSidesCBR2019-rescue:Conn_02x03_Odd_Even
- J3: symbol CONN_01X08 -> BSidesCBR2019-rescue:CONN_01X08
- R1, R2, R3, R4, R5, R6: symbol R_Small -> BSidesCBR2019-rescue:R_Small
- SW1, SW3, SW4, SW5: symbol SW_Push -> BSidesCBR2019-rescue:SW_Push
- SW2: symbol SW_SPDT -> BSidesCBR2019-rescue:SW_SPDT
- U1: symbol ATMEGA328P-AU -> BSidesCBR2019-rescue:ATMEGA328P-AU
- U2: symbol Nokia_5110_LCD -> BSidesCBR2019-rescue:Nokia_5110_LCD
- Y1: symbol Crystal_GND24 -> BSidesCBR2019-rescue:Crystal_GND24
Connections:
- net D3 is gone; now on net BUTTONOK: U1.1 ((PCINT19/OC2B/INT1)PD3)
- net D4 is gone; now on net BUTTONR: U1.2 ((PCINT20/XCK/T0)PD4)
- net BUTTONL: now reaches SW3.2
- net BUTTONL: now also U1.32 ((PCINT18/INT0)PD2)
- net BUTTONOK: now reaches SW4.2
- net BUTTONS renamed BUTTONR
- net BUTTONR: no longer U1.32 ((PCINT18/INT0)PD2)

Commit message: Added footprints and models, v8 gerbs
Parts:
- BT1: symbol BSidesCBR2019-rescue:Battery_Cell_PWR -> BSidesCBR2019-rescue:Battery_Cell_PWR-BSidesCBR2019-rescue
- C1: symbol BSidesCBR2019-rescue:C_Small -> BSidesCBR2019-rescue:C_Small-BSidesCBR2019-rescue
- D1, D2, D3, D4: symbol BSidesCBR2019-rescue:LED_Small -> BSidesCBR2019-rescue:LED_Small-BSidesCBR2019-rescue
- J1: symbol BSidesCBR2019-rescue:Conn_02x02_Odd_Even -> BSidesCBR2019-rescue:Conn_02x02_Odd_Even-BSidesCBR2019-rescue
- J2: symbol BSidesCBR2019-rescue:Conn_02x03_Odd_Even -> BSidesCBR2019-rescue:Conn_02x03_Odd_Even-BSidesCBR2019-rescue
- J3: symbol BSidesCBR2019-rescue:CONN_01X08 -> BSidesCBR2019-rescue:CONN_01X08-BSidesCBR2019-rescue
- R1, R2, R3, R4, R5, R6: symbol BSidesCBR2019-rescue:R_Small -> BSidesCBR2019-rescue:R_Small-BSidesCBR2019-rescue
- SW1: symbol BSidesCBR2019-rescue:SW_Push -> BSidesCBR2019-rescue:SW_Push-BSidesCBR2019-rescue
- SW2: footprint Buttons_Switches_SMD:SW_SPDT_PCM12 -> Button_Switch_SMD:SW_SPDT_PCM12; symbol BSidesCBR2019-rescue:SW_SPDT -> BSidesCBR2019-rescue:SW_SPDT-BSidesCBR2019-rescue
- SW3, SW4, SW5: footprint Buttons_Switches_SMD:SW_SPST_B3SL-1002P -> Button_Switch_SMD:SW_SPST_B3SL-1002P; symbol BSidesCBR2019-rescue:SW_Push -> BSidesCBR2019-rescue:SW_Push-BSidesCBR2019-rescue
- U1: symbol BSidesCBR2019-rescue:ATMEGA328P-AU -> BSidesCBR2019-rescue:ATMEGA328P-AU-BSidesCBR2019-rescue
- U2: symbol BSidesCBR2019-rescue:Nokia_5110_LCD -> BSidesCBR2019-rescue:Nokia_5110_LCD-BSidesCBR2019-rescue
- Y1: symbol BSidesCBR2019-rescue:Crystal_GND24 -> BSidesCBR2019-rescue:Crystal_GND24-BSidesCBR2019-rescue
Connections:
- net +3V3: no longer SW3.1, SW4.1, SW5.1
- net GND: now also SW3.1, SW4.1, SW5.1
Changed lines of the file:
@@
 $EndDescr
 $Comp
-L BSidesCBR2019-rescue:ATMEGA328P-AU U1
+L BSidesCBR2019-rescue:ATMEGA328P-AU-BSidesCBR2019-rescue U1
 U 1 1 5B1519FE
 P 3100 2500
@@
 $EndComp
 $Comp
-L BSidesCBR2019-rescue:Crystal_GND24 Y1
+L BSidesCBR2019-rescue:Crystal_GND24-BSidesCBR2019-rescue Y1
 U 1 1 5B1596CA
 P 4950 2250
@@
 $EndComp
 $Comp
-L BSidesCBR2019-rescue:R_Small R1
+L BSidesCBR2019-rescue:R_Small-BSidesCBR2019-rescue R1
 U 1 1 5B15A6E6
 P 4750 2150
@@
 $EndComp
 $Comp
-L BSidesCBR2019-rescue:SW_Push SW1
+L BSidesCBR2019-rescue:SW_Push-BSidesCBR2019-rescue SW1
 U 1 1 5B15C0ED
 P 7000 5100
@@
 $EndComp
 $Comp
-L BSidesCBR2019-rescue:Conn_02x03_Odd_Even J2
+L BSidesCBR2019-rescue:Conn_02x03_Odd_Even-BSidesCBR2019-rescue J2
 U 1 1 5B15C48C
 P 7200 4550
@@
 $EndComp
 $Comp
-L BSidesCBR2019-rescue:R_Small R4
+L BSidesCBR2019-rescue:R_Small-BSidesCBR2019-rescue R4
 U 1 1 5B15CE2B
 P 6750 4100
@@
 GND
 $Comp
-L BSidesCBR2019-rescue:Nokia_5110_LCD U2
+L BSidesCBR2019-rescue:Nokia_5110_LCD-BSidesCBR2019-rescue U2
 U 1 1 5B1626A2
 P 6550 1550
@@
 LCDBL+
 $Comp
-L BSidesCBR2019-rescue:LED_Small D1
+L BSidesCBR2019-rescue:LED_Small-BSidesCBR2019-rescue D1
 U 1 1 5B16F4CE
 P 5650 2400
@@
 $EndComp
 $Comp
-L BSidesCBR2019-rescue:LED_Small D2
+L BSidesCBR2019-rescue:LED_Small-BSidesCBR2019-rescue D2
 U 1 1 5B16F558
 P 5650 2750
@@
 TXD
 $Comp
-L BSidesCBR2019-rescue:Battery_Cell_PWR BT1
+L BSidesCBR2019-rescue:Battery_Cell_PWR-BSidesCBR2019-rescue BT1
 U 1 1 5B180D41
 P 850 2300
@@
 TXD
 $Comp
-L BSidesCBR2019-rescue:Conn_02x02_Odd_Even J1
+L BSidesCBR2019-rescue:Conn_02x02_Odd_Even-BSidesCBR2019-rescue J1
 U 1 1 5B7A0349
 P 7500 4100
@@
 $EndComp
 $Comp
-L BSidesCBR2019-rescue:R_Small R5
+L BSidesCBR2019-rescue:R_Small-BSidesCBR2019-rescue R5
 U 1 1 5B7A725B
 P 5850 2750
@@
 $EndComp
 $Comp
-L BSidesCBR2019-rescue:LED_Small D3
+L BSidesCBR2019-rescue:LED_Small-BSidesCBR2019-rescue D3
 U 1 1 5BA8E247
 P 5650 3100
@@
 $EndComp
 $Comp
-L BSidesCBR2019-rescue:LED_Small D4
+L BSidesCBR2019-rescue:LED_Small-BSidesCBR2019-rescue D4
 U 1 1 5BA8E357
 P 5650 3450
@@
 $EndComp
 $Comp
-L BSidesCBR2019-rescue:R_Small R3
+L BSidesCBR2019-rescue:R_Small-BSidesCBR2019-rescue R3
 U 1 1 5BA8E4CA
 P 5850 3100
@@
 $EndComp
 $Comp
-L BSidesCBR2019-rescue:R_Small R6
+L BSidesCBR2019-rescue:R_Small-BSidesCBR2019-rescue R6
 U 1 1 5BA8E550
 P 5850 3450
@@
 $EndComp
 $Comp
-L BSidesCBR2019-rescue:R_Small R2
+L BSidesCBR2019-rescue:R_Small-BSidesCBR2019-rescue R2
 U 1 1 5BA8E5DF
 P 5850 2400
@@
 $EndComp
 $Comp
-L BSidesCBR2019-rescue:C_Small C1
+L BSidesCBR2019-rescue:C_Small-BSidesCBR2019-rescue C1
 U 1 1 5BA8FEB5
 P 5900 1250
@@
 	4100 3400 4200 3400
 $Comp
-L BSidesCBR2019-rescue:CONN_01X08 J3
+L BSidesCBR2019-rescue:CONN_01X08-BSidesCBR2019-rescue J3
 U 1 1 5BD855DB
 P 4600 5250
@@
 	4200 5600 4400 5600
 $Comp
-L BSidesCBR2019-rescue:SW_SPDT SW2
+L BSidesCBR2019-rescue:SW_SPDT-BSidesCBR2019-rescue SW2
 U 1 1 5BD88412
 P 950 1650
-F 0 "SW2" H 950 1775 50  0000 C CNN
+F 0 "SW2" H 950 1850 50  0000 C CNN
 F 1 "SW_SPST" H 950 1450 50  0000 C CNN
-F 2 "Buttons_Switches_SMD:SW_SPDT_PCM12" H 950 1650 50  0001 C CNN
+F 2 "Button_Switch_SMD:SW_SPDT_PCM12" H 950 1650 50  0001 C CNN
 F 3 "" H 950 1650 50  0001 C CNN
 	1    950  1650
@@
 BAT+
 $Comp
-L BSidesCBR2019-rescue:SW_Push SW3
+L BSidesCBR2019-rescue:SW_Push-BSidesCBR2019-rescue SW3
 U 1 1 5BD89C01
 P 4900 4150
 F 0 "SW3" H 4950 4250 50  0000 L CNN
 F 1 "<<" H 4900 4090 50  0000 C CNN
-F 2 "Buttons_Switches_SMD:SW_SPST_B3SL-1002P" H 4900 4350 50  0001 C CNN
+F 2 "Button_Switch_SMD:SW_SPST_B3SL-1002P" H 4900 4350 50  0001 C CNN
 F 3 "" H 4900 4350 50  0001 C CNN
 	1    4900 4150
@@
 $EndComp
 $Comp
-L BSidesCBR2019-rescue:SW_Push SW4
+L BSidesCBR2019-rescue:SW_Push-BSidesCBR2019-rescue SW4
 U 1 1 5BD89EFA
 P 5300 4150
 F 0 "SW4" H 5350 4250 50  0000 L CNN
 F 1 "O" H 5300 4090 50  0000 C CNN
-F 2 "Buttons_Switches_SMD:SW_SPST_B3SL-1002P" H 5300 4350 50  0001 C CNN
+F 2 "Button_Switch_SMD:SW_SPST_B3SL-1002P" H 5300 4350 50  0001 C CNN
 F 3 "" H 5300 4350 50  0001 C CNN
 	1    5300 4150
@@
 $EndComp
 $Comp
-L BSidesCBR2019-rescue:SW_Push SW5
+L BSidesCBR2019-rescue:SW_Push-BSidesCBR2019-rescue SW5
 U 1 1 5BD89F58
 P 5700 4150
 F 0 "SW5" H 5750 4250 50  0000 L CNN
 F 1 ">>" H 5700 4090 50  0000 C CNN
-F 2 "Buttons_Switches_SMD:SW_SPST_B3SL-1002P" H 5700 4350 50  0001 C CNN
+F 2 "Button_Switch_SMD:SW_SPST_B3SL-1002P" H 5700 4350 50  0001 C CNN
 F 3 "" H 5700 4350 50  0001 C CNN
 	1    5700 4150
 	0    1    1    0
 $EndComp
-Text GLabel 5300 3800 1    60   Input ~ 0
-+3.3v
 Wire Wire Line
 	4900 3950 4900 3850
@@
 Wire Wire Line
 	5700 3850 5700 3950
-Wire Wire Line
-	5300 3800 5300 3850
 Connection ~ 5300 3850
 Wire Wire Line
@@
 Wire Wire Line
 	4900 4700 4900 4350
+$Comp
+L power:GND #PWR0101
+U 1 1 5C149655
+P 5300 3700
+F 0 "#PWR0101" H 5300 3450 50  0001 C CNN
+F 1 "GND" H 5300 3550 50  0000 C CNN
+F 2 "" H 5300 3700 50  0001 C CNN
+F 3 "" H 5300 3700 50  0001 C CNN
+	1    5300 3700
+	-1   0    0    1
+$EndComp
+Wire Wire Line
+	5300 3700 5300 3850
 $EndSCHEMATC
